Commit message: 카메라 두대달았지만 namespace규칙어김

File: champ_description/urdf/accessories.urdf.xacro (robot description, xacro)
@@ -16,6 +16,11 @@
         <xacro:asus_camera
             parent="${base_name}"
-            name="camera">
+            name="champ_front">
             <origin xyz="${base_length / 2} 0.0 -${base_height / 2 + 0.01}" rpy="0 0 0"/>
+        </xacro:asus_camera>
+        <xacro:asus_camera
+            parent="${base_name}"
+            name="champ_rear">
+            <origin xyz="${base_length / 2} 0.0 -${base_height / 2 + 0.01}" rpy="0 0 1.570"/>
         </xacro:asus_camera>
         <link name="imu_link">
@@ -65,8 +70,9 @@
                 </sensor>
             </gazebo>
-        <xacro:include filename="$(find velodyne_description)/urdf/VLP-16.urdf.xacro"/>
-        <xacro:VLP-16 parent="${base_name}" name="champ" topic="velodyne_points" hz="10" samples="1024" gpu="false" lasers="16" max_range="100">
+        <!-- original code -->
+        <!-- <xacro:include filename="$(find velodyne_description)/urdf/VLP-16.urdf.xacro"/>
+        <xacro:VLP-16 parent="${base_name}" name="velodyne" topic="velodyne_points" hz="10" samples="1024" gpu="false" lasers="16" max_range="100">
             <origin xyz="0 0 ${base_height / 2}" rpy="0 0 0" />
-        </xacro:VLP-16>
+        </xacro:VLP-16> -->
         <!-- <xacro:include filename="$(find champ_arm_description)/urdf/champ_arm.urdf.xacro" />
         <xacro:champ_arm parent="${base_name}">

Commit message: namespace정리완료 벨로다인달기 남음

File: champ_description/urdf/accessories.urdf.xacro (robot description, xacro)
@@ -16,10 +16,12 @@
         <xacro:asus_camera
             parent="${base_name}"
-            name="champ_front">
+            name="front_camera"
+            robotname="champ">
             <origin xyz="${base_length / 2} 0.0 -${base_height / 2 + 0.01}" rpy="0 0 0"/>
         </xacro:asus_camera>
         <xacro:asus_camera
             parent="${base_name}"
-            name="champ_rear">
+            name="rear_camera"
+            robotname="champ">
             <origin xyz="${base_length / 2} 0.0 -${base_height / 2 + 0.01}" rpy="0 0 1.570"/>
         </xacro:asus_camera>

File: champ_description/urdf/asus_camera.urdf.xacro (robot description, xacro)
@@ -68,5 +68,5 @@
      the openni gazebo plugin.
     -->
-    <xacro:macro name="asus_camera" params="name parent *origin">
+    <xacro:macro name="asus_camera" params="name robotname parent *origin">
       <xacro:asus_camera_model name="${name}" parent="${parent}">
         <xacro:insert_block name="origin" />
@@ -94,6 +94,6 @@
           <plugin name="${name}_camera_controller" filename="libgazebo_ros_camera.so">
             <ros>
-              <!-- <namespace>custom_ns</namespace> -->
-              <argument>custom_camera/image_raw:=${name}/rgb/image_raw</argument>
+              <namespace>${robotname}</namespace>
+              <argument>custom_camera/image_raw:=/${name}/rgb/image_raw</argument>
               <argument>custom_camera/image_depth:=${name}/depth/image_raw</argument>
               <argument>custom_camera/camera_info:=custom_camera/custom_info_raw</argument>

Commit message: test:

File: champ_description/urdf/accessories.urdf.xacro (robot description, xacro)
@@ -1,8 +1,12 @@
 <?xml version="1.0"?>
 <robot xmlns:xacro="http://ros.org/wiki/xacro">
-    <xacro:macro name="accessories" params="base_name base_length base_height  " >
-        <xacro:include filename="$(find champ_description)/urdf/hokuyo_utm30lx.urdf.xacro" />
+    <xacro:macro name="accessories" params="base_name base_length base_height ssafyname" >
+        <!-- <xacro:include filename="$(find champ_description)/urdf/hokuyo_utm30lx.urdf.xacro" /> -->
         <xacro:include filename="$(find champ_description)/urdf/asus_camera.urdf.xacro" />
-        <xacro:hokuyo_utm30lx
+        <xacro:include filename="$(find velodyne_description)/urdf/VLP-16.urdf.xacro"/>
+        <!-- <xacro:VLP-16 parent="${base_name}" name="${ssafyname}" topic="velodyne_points" hz="10" samples="1024" gpu="false" lasers="16" max_range="100">
+            <origin xyz="0 0 ${base_height+10}" rpy="0 0 0" />
+        </xacro:VLP-16> -->
+        <!-- <xacro:hokuyo_utm30lx
             name="hokuyo"
             parent="${base_name}"
@@ -13,9 +17,9 @@
             max_angle="-130" >
             <origin xyz="0.0 0.0 ${base_height / 2 + 0.04}" rpy="0 0 0"/>
-        </xacro:hokuyo_utm30lx>
+        </xacro:hokuyo_utm30lx> -->
         <xacro:asus_camera
             parent="${base_name}"
             name="front_camera"
-            robotname="champ">
+            robotname="${ssafyname}">
             <origin xyz="${base_length / 2} 0.0 -${base_height / 2 + 0.01}" rpy="0 0 0"/>
         </xacro:asus_camera>
@@ -23,8 +27,15 @@
             parent="${base_name}"
             name="rear_camera"
-            robotname="champ">
+            robotname="${ssafyname}">
             <origin xyz="${base_length / 2} 0.0 -${base_height / 2 + 0.01}" rpy="0 0 1.570"/>
         </xacro:asus_camera>
         <link name="imu_link">
+            <inertial>
+                <mass value="0.001"/>
+                <origin xyz="0 0 0" rpy="0 0 0"/>
+                <inertia ixx="1e-09" ixy="0.0" ixz="0.0" iyy="1e-09" iyz="0.0" izz="1e-09"/>
+            </inertial>
+        </link>
+        <link name ="gps_link">
             <inertial>
                 <mass value="0.001"/>
@@ -37,43 +48,45 @@
             <child link="imu_link" />
         </joint>
+        <joint name="gps_joint" type="fixed">
+            <parent link="${base_name}" />
+            <child link="gps_link" />
+        </joint>
         <gazebo reference="imu_link">
-                <sensor name="imu_controller" type="imu">
-                    <always_on>true</always_on>
-                    <update_rate>100</update_rate>
-                    <plugin name="gazebo_ros_imu_sensor" filename="libgazebo_ros_imu_sensor.so">
-                        <ros>
-                            <namespace>champ</namespace>
-                            <argument>~/out:=imu</argument>
-                        </ros>
-                        <!-- <updateRate>50.0</updateRate>
-                        <bodyName>imu_link</bodyName>
-                        <topicName>imu/data</topicName>
-                        <accelDrift>0.005 0.005 0.005</accelDrift>
-                        <accelGaussianNoise>0.005 0.005 0.005</accelGaussianNoise>
-                        <rateDrift>0.005 0.005 0.005 </rateDrift>
-                        <rateGaussianNoise>0.005 0.005 0.005 </rateGaussianNoise>
-                        <headingDrift>0.005</headingDrift>
-                        <headingGaussianNoise>0.005</headingGaussianNoise> -->
-                    </plugin>
-                </sensor>
-                <sensor name="champ_gps" type="gps">
-                    <!-- 센서 기본 설정 -->
-                    <always_on>true</always_on>
-                    <update_rate>8</update_rate> <!-- 초당 8회 업데이트 예시 -->
-                    <!-- Gazebo ROS GPS 플러그인 -->
-                    <plugin name="my_gps_plugin" filename="libgazebo_ros_gps_sensor.so">
+            <sensor name="imu_controller" type="imu">
+                <always_on>true</always_on>
+                <update_rate>100</update_rate>
+                <plugin name="gazebo_ros_imu_sensor" filename="libgazebo_ros_imu_sensor.so">
                     <ros>
-                        <!-- 네임스페이스 설정 -->
-                        <namespace>champ</namespace>
-                        <remapping>~/out:=gps</remapping>
+                        <namespace>${ssafyname}</namespace>
+                        <argument>~/out:=imu</argument>
                     </ros>
-                    <!-- 아래 항목들은 플러그인에 따라 다르나, 일반적으로 설정 -->
-                    </plugin>
-                </sensor>
-            </gazebo>
+                    <!-- <updateRate>50.0</updateRate>
+                    <bodyName>imu_link</bodyName>
+                    <topicName>imu/data</topicName>
+                    <accelDrift>0.005 0.005 0.005</accelDrift>
+                    <accelGaussianNoise>0.005 0.005 0.005</accelGaussianNoise>
+                    <rateDrift>0.005 0.005 0.005 </rateDrift>
+                    <rateGaussianNoise>0.005 0.005 0.005 </rateGaussianNoise>
+                    <headingDrift>0.005</headingDrift>
+                    <headingGaussianNoise>0.005</headingGaussianNoise> -->
+                </plugin>
+            </sensor>
+        </gazebo>
+        <gazebo reference="gps_link">
+            <sensor name="gps_controller" type="gps">
+                <always_on>true</always_on>
+                <update_rate>100</update_rate>
+                <plugin name="gazebo_ros_gps" filename="libgazebo_ros_gps.so">
+                    <ros>
+                        <namespace>${ssafyname}</namespace>
+                        <argument>~/fix:=fix</argument>
+                    </ros>
+                </plugin>
+            </sensor>
+        </gazebo>
         <!-- original code -->
-        <!-- <xacro:include filename="$(find velodyne_description)/urdf/VLP-16.urdf.xacro"/>
-        <xacro:VLP-16 parent="${base_name}" name="velodyne" topic="velodyne_points" hz="10" samples="1024" gpu="false" lasers="16" max_range="100">
-            <origin xyz="0 0 ${base_height / 2}" rpy="0 0 0" />
+            <!-- <xacro:include filename="$(find velodyne_description)/urdf/VLP-16.urdf.xacro"/>
+        <xacro:VLP-16 parent="${base_name}" name="my3dlidar" topic="velodyne_points" hz="10" samples="1024" gpu="false" lasers="16" max_range="100">
+            <origin xyz="0 0 ${base_height}" rpy="0 0 0" />
         </xacro:VLP-16> -->
         <!-- <xacro:include filename="$(find champ_arm_description)/urdf/champ_arm.urdf.xacro" />

File: champ_description/urdf/champ.urdf.xacro (robot description, xacro)
@@ -46,4 +46,5 @@
         base_length="${base_x_length}"
         base_height="${base_z_length}"
+        ssafyname="champ"
     />
     <xacro:champ_leg leg="lf"/>
